Commit message: feat: realistic UR5e URDF and Dashboard 2 arm plus pendant
Replace the primitive viewer with vendored UR5e STL meshes (BSD-3-Clause)
and add ui-robot-arm and ui-robot-controller so the 3D view and teach
pendant render on a FlowFuse Dashboard 2 page. Package name is
node-red-dashboard-2-robot-arm so Dashboard can discover the widgets.

File: models/ur5e/ur5e.urdf (robot description, URDF)
Before this commit: robot ur5e_gripper, 13 links, 12 joints
Links:
- removed link finger_left_link
- removed link finger_right_link
- removed link gripper_base_link
Joints:
- removed joint finger_joint
- removed joint finger_joint_right
- removed joint gripper_fixed
